File: untitled.kicad_sch (KiCad schematic)
At the start: 1 part, among them U1 MSP430FR4133IPMR

Commit message: edit mspADC
Parts:
- U1: footprint MSP430FR4133IPMR:QFP50P1200X1200X160-64N -> Package_QFP:LQFP-64-MSP430FR4133-PM0064A_N
